Commit message: repair simulation 1/2

File: simulation/models/m_robot/m_robot.xacro (robot description, xacro)
@@ -2,15 +2,15 @@
 <robot name="robot" xmlns:xacro="http://www.ros.org/wiki/xacro">
   <xacro:property name="PI" value="3.1415926535897931"/>
-  <xacro:property name="chassisHeight" value="0.1"/>
-  <xacro:property name="chassisLength" value="0.4"/>
-  <xacro:property name="chassisWidth" value="0.4"/>
+  <xacro:property name="chassisHeight" value="0.05"/>
+  <xacro:property name="chassisLength" value="0.2"/>
+  <xacro:property name="chassisWidth" value="0.2"/>
   <xacro:property name="chassisMass" value="50"/>
-  <xacro:property name="casterRadius" value="0.05"/>
+  <xacro:property name="casterRadius" value="0.02"/>
   <xacro:property name="casterMass" value="5"/>
-  <xacro:property name="wheelWidth" value="0.05"/>
-  <xacro:property name="wheelRadius" value="0.1"/>
-  <xacro:property name="wheelPos" value="0.2"/>
+  <xacro:property name="wheelWidth" value="0.02"/>
+  <xacro:property name="wheelRadius" value="0.05"/>
+  <xacro:property name="wheelPos" value="0.1"/>
   <xacro:property name="wheelMass" value="5"/>
-  <xacro:property name="rplidarMass" value="0.170"/>
+  <xacro:property name="rplidarMass" value="0.17"/>
   <xacro:property name="rplidarSamples" value="1020"/>
   <xacro:property name="rplidarResolution" value="1"/>
@@ -18,5 +18,5 @@
   <xacro:property name="rplidarMaxAngle" value="6.283185307"/>
   <xacro:property name="rplidarRange" value="12"/>
-  <xacro:property name="rplidarLaserHeight" value="0.03" />
+  <xacro:property name="rplidarLaserHeight" value="0.04" />
   <xacro:include filename="$(find simulation)/models/m_robot/m_robot.gazebo" />
   <xacro:include filename="$(find simulation)/models/m_robot/materials.xacro" />
@@ -43,7 +43,7 @@
     </visual>
     <inertial>
-      <origin xyz="0 0 ${wheelRadius}" rpy="0 0 0"/>
+      <origin xyz="0 0 ${wheelRadius/2}" rpy="0 0 0"/>
       <mass value="${chassisMass}"/>
-      <box_inertia m="${chassisMass}" x="${chassisLength}" y="${chassisWidth}" z="${chassisHeight}"/>
+      <box_inertia m="${chassisMass}" x="${chassisWidth}" y="${chassisLength}" z="${chassisHeight}"/>
     </inertial>
   </link>
@@ -98,5 +98,5 @@
     <parent link="chassis"/>
     <child link="rplidar"/>
-    <origin xyz="${-casterRadius+chassisLength/2} 0 ${casterRadius+chassisHeight + rplidarLaserHeight}" rpy="0 0 0" />
+    <origin xyz="${-2*casterRadius+chassisLength/2} 0 ${casterRadius+chassisHeight + rplidarLaserHeight}" rpy="0 0 0" />
     <axis xyz="0 1 0" />
   </joint>

File: simulation/models/m_robot/macros.xacro (robot description, xacro)
@@ -7,7 +7,7 @@
       </macro>
       <macro name="box_inertia" params="m x y z">
-        <inertia  ixx="${m*(y*y+z*z)/12}" ixy = "0" ixz = "0"
-                  iyy="${m*(x*x+z*z)/12}" iyz = "0"
-                  izz="${m*(x*x+z*z)/12}" />
+        <inertia  iyy="${m*(y*y+z*z)/12}" ixy = "0" ixz = "0"
+                  izz="${m*(x*x+y*y)/12}" iyz = "0"
+                  ixx="${m*(x*x+z*z)/12}" />
       </macro>
       <macro name="sphere_inertia" params="m r">
@@ -30,16 +30,16 @@
             <cylinder length="${wheelWidth}" radius="${wheelRadius}"/>
           </geometry>
-          <surface>
-            <friction>
+          <!--<surface>
+           <friction>
               <ode>
-                <mu>1000000</mu>
-                <mu2>1000000</mu2>
-                <!--<kp  value="1000"/>
-                <kd  value="100" />-->
-                <minDepth>0.001</minDepth>
-                <maxVel>0.01</maxVel>
+                <mu1 value="100000000" />
+                <mu2 value="100000000" />
+                <kp  value="100000000"/>
+                <kd  value="100" />
+                <minDepth>0.01</minDepth>
+                <maxVel>0.001</maxVel>
               </ode>
             </friction>
-          </surface>
+          </surface>-->
         </collision>
         <inertial>
@@ -51,10 +51,10 @@
         <gazebo reference="${lr}_wheel">
           <material>Gazebo/Black</material>
-          <mu1 value="1000000"/>
-          <mu2 value="1000000"/>
-         <!-- <kp value="1000"/>
-          <kd value="100" />-->
-          <minDepth>0.001</minDepth>
-          <maxVel>0.01</maxVel>
+          <mu1 value="100000000000"/>
+          <mu2 value="100000000000"/>
+          <kp value="10000000"/>
+          <kd value="0" />
+          <minDepth>0.000001</minDepth>
+          <maxVel>0.0001</maxVel>
         </gazebo>
        <joint name="${lr}_wheel_hinge" type="continuous">

Commit message: repair model

File: simulation/models/m_robot/m_robot.xacro (robot description, xacro)
@@ -22,5 +22,26 @@
   <xacro:include filename="$(find simulation)/models/m_robot/materials.xacro" />
   <xacro:include filename="$(find simulation)/models/m_robot/macros.xacro" />
-  <link name="m_robot"/>
+  <link name="m_robot">
+      <inertial>
+        <mass value="0.0001" />
+        <origin xyz="0 0 0" />
+        <inertia ixx="0.0001" ixy="0.0" ixz="0.0"
+                 iyy="0.0001" iyz="0.0"
+                 izz="0.0001" />
+      </inertial>
+      <visual>
+          <origin xyz="0 0 0" rpy="0 0 0" />
+          <geometry>
+              <box size="0.001 0.001 0.001" />
+          </geometry>
+          <material name="Green" />
+      </visual>
+      <collision>
+          <origin xyz="0 0 0.128" rpy="0 0 0" />
+          <geometry>
+            <box size="0.001 0.001 0.001" />
+          </geometry>
+      </collision>
+  </link>
   <joint name="base_joint" type="fixed">
     <parent link="m_robot"/>

File: simulation/models/m_robot/macros.xacro (robot description, xacro)
@@ -30,16 +30,4 @@
             <cylinder length="${wheelWidth}" radius="${wheelRadius}"/>
           </geometry>
-          <!--<surface>
-           <friction>
-              <ode>
-                <mu1 value="100000000" />
-                <mu2 value="100000000" />
-                <kp  value="100000000"/>
-                <kd  value="100" />
-                <minDepth>0.01</minDepth>
-                <maxVel>0.001</maxVel>
-              </ode>
-            </friction>
-          </surface>-->
         </collision>
         <inertial>
@@ -51,10 +39,8 @@
         <gazebo reference="${lr}_wheel">
           <material>Gazebo/Black</material>
-          <mu1 value="100000000000"/>
-          <mu2 value="100000000000"/>
-          <kp value="10000000"/>
-          <kd value="0" />
-          <minDepth>0.000001</minDepth>
-          <maxVel>0.0001</maxVel>
+            <mu1 value="100.0" />
+            <mu2 value="100.0" />
+            <kp  value="1000000.0" />
+            <kd  value="1.0" />
         </gazebo>
        <joint name="${lr}_wheel_hinge" type="continuous">
